File: nixieclock/power.kicad_sch (KiCad schematic)
At the start: 10 parts, among them J1 USB_C_Receptacle_USB2.0_14P, Q1 PMOS, U1 AMS1117-3.3, U2 HUSB238_002DD

Commit message: High Voltage!
Parts:
- added C15: 100uF, symbol Device:C_Polarized_US
- added C16, C17: 100nF, symbol Device:C
- added C18: 4.7uF >250V, symbol Device:C_Polarized_US
- added C19: 100nF >250V, symbol Device:C
- added D1: ES2F-E3/52T, symbol Device:D
- added L1: 100uH (2A), symbol Device:L
- added Q2: STD17NF25, lcsc:TO-252-3_L6.5-W5.8-P4.58-TL, symbol lcsc:STD17NF25
- added R10: 1.3M, symbol Device:R
- added R11: 11.57k, symbol Device:R
- added R9: 0.05, symbol Device:R
- added TP1: TestPoint, symbol Connector:TestPoint
- added U5: MAX1771xSA, Package_SO:SO-8_3.9x4.9mm_P1.27mm, symbol Regulator_Switching:MAX1771xSA
Connections:
- net +12V: now also C15.1, C16.1, L1.1, U5.2 (V+)
- net GND: now also C15.2, C16.2, C17.2, C18.2, C19.2, R11.2, R9.2, U5.6 (AGND), U5.7 (GND)
- new net: Q2.3 (S), R9.1, U5.8 (CS)
- new net: D1.2 (A), L1.2, Q2.2 (D)
- new net: C17.1, U5.5 (REF)
- new net: Q2.1 (G), U5.1 (EXT)
- new net +170V: C18.1, C19.1, D1.1 (K), R10.1, TP1.1
- new net MAX1771_EN: U5.4 (SHDN)
- new net MAX1771_FB: R10.2, R11.1, U5.3 (FB)
Other:
- note added: "This should be 170 Volts, but we should do a test and block power unless it's correct"
